Commit message: added rs camera to gr1t1

File: GRX/GR1/GR1T1/urdf/GR1T1_inspire_hand.urdf (robot description, URDF)
Before this commit: robot GR1T1_inspire_hand, 73 links, 72 joints
Links:
- added link realsense_bottom_screw_frame
- added link realsense_cam; visual mesh filename=../meshes/d435_1.stl
- added link realsense_color_frame
- added link realsense_color_optical_frame; visual sphere radius=0.008
- added link realsense_depth_frame
- added link realsense_depth_optical_frame; visual sphere radius=0.008
Joints:
- added joint realsense_color_joint: type fixed, parent realsense_cam, child realsense_color_frame, origin xyz=-0.025 0.015 0 rpy=0 0 0
- added joint realsense_color_optical_joint: type fixed, parent realsense_color_frame, child realsense_color_optical_frame, origin xyz=0 0 0 rpy=-1.5707963267948966 0 -1.5707963267948966
- added joint realsense_depth_joint: type fixed, parent realsense_cam, child realsense_depth_frame, origin xyz=0 0 0 rpy=0 0 0
- added joint realsense_depth_optical_joint: type fixed, parent realsense_depth_frame, child realsense_depth_optical_frame, origin xyz=0 0 0 rpy=-1.5707963267948966 0 -1.5707963267948966
- added joint realsense_joint: type fixed, parent head_pitch_link, child realsense_bottom_screw_frame, origin xyz=0.06682 0 -0.02137 rpy=0 0 0
- added joint realsense_link_joint: type fixed, parent realsense_bottom_screw_frame, child realsense_cam, origin xyz=0.0106 0.0175 0.0 rpy=0 0 0
